File: PCB_v1.kicad_sch (KiCad schematic)
At the start: 4 parts, among them J1 Conn_01x14_Female, U1 ESP32-DEVKIT-V1, U2 OV7670

Commit message: working on power circuit
Parts:
- removed F1: Fuse, symbol Device:Fuse
- added C?: 10uF, Capacitor_THT:C_Rect_L7.2mm_W8.5mm_P5.00mm_FKP2_FKP2_MKS2_MKP2, symbol Device:C
- added D?: LED, LED_THT:LED_D1.8mm_W3.3mm_H2.4mm, symbol Device:LED
- added F?: Fuse, ProjectLibraries:fuse_tht, symbol Device:Fuse
- added H? (x10): MountingHole, symbol Mechanical:MountingHole
- added J?: +5V, symbol Connector:Conn_01x01_Female
- added J?: +3.3V, symbol Connector:Conn_01x01_Female
- added J? (x2): GND, symbol Connector:Conn_01x01_Female
- added J?: PowerInput5V, symbol Connector:Conn_01x02_Female
- added R?: 500, Resistor_THT:R_Axial_DIN0207_L6.3mm_D2.5mm_P10.16mm_Horizontal, symbol Device:R
- added SW?: SW_SPDT, Button_Switch_THT:SW_E-Switch_EG1224_SPDT_Angled, symbol Switch:SW_SPDT
- added TP? (x3): TestPoint, symbol Connector:TestPoint
Connections:
- new net: F?.1, J?.1 (Pin_1)
- new net: F?.2, SW?.2 (B)
- new net: D?.2 (A), R?.2
- new net +3.3V: J?.1 (Pin_1), TP?.1
- new net +5V: C?.1, J?.1 (Pin_1), R?.1, SW?.1 (A), TP?.1
- new net GND: C?.2, D?.1 (K), J?.1 (Pin_1), J?.1 (Pin_1), J?.2 (Pin_2), TP?.1
- no-connect marks 0 -> 1

Commit message: schematic done
Parts:
- removed J1: Conn_01x14_Female, symbol Connector:Conn_01x14_Female
- removed J?: +5V, symbol Connector:Conn_01x01_Female
- removed J?: +3.3V, symbol Connector:Conn_01x01_Female
- removed J? (x2): GND, symbol Connector:Conn_01x01_Female
- removed TP?: TestPoint, symbol Connector:TestPoint
- removed U1: ESP32-DEVKIT-V1, ESP32-DEVKIT-V1:MODULE_ESP32_DEVKIT_V1, symbol ESP32-DEVKIT-V1:ESP32-DEVKIT-V1
- removed U2: OV7670, OV7670:OV7670, symbol OV7670:OV7670
- added C?: 100uF, Capacitor_THT:C_Rect_L7.2mm_W8.5mm_P5.00mm_FKP2_FKP2_MKS2_MKP2, symbol Device:C
- added C?: 10uF, Capacitor_THT:C_Rect_L7.2mm_W8.5mm_P5.00mm_FKP2_FKP2_MKS2_MKP2, symbol Device:C
- added C?: 1000uF, Capacitor_THT:C_Rect_L7.2mm_W8.5mm_P5.00mm_FKP2_FKP2_MKS2_MKP2, symbol Device:C
- added D?: LED, LED_THT:LED_D1.8mm_W3.3mm_H2.4mm, symbol Device:LED
- added J?: StepperSignals, symbol Connector:Conn_01x02_Male
- added J?: LogicShifterOut, symbol Connector:Conn_01x06_Female
- added J?: LogicShifterIn, symbol Connector:Conn_01x06_Female
- added J?: StepperGND, symbol Connector:Conn_01x02_Female
- added J?: PowerOutput11.1V, symbol Connector:Conn_01x02_Female
- added J?: Thermistor, symbol Connector:Conn_01x02_Male
- added J?: PowerInput11.1V, symbol Connector:Screw_Terminal_01x02
- added R?: 100k, symbol Device:R
- added R?: 500, Resistor_THT:R_Axial_DIN0207_L6.3mm_D2.5mm_P10.16mm_Horizontal, symbol Device:R
- added SW?: SW_SPDT, Button_Switch_THT:SW_E-Switch_EG1224_SPDT_Angled, symbol Switch:SW_SPDT
- added TP? (x5): TestPoint, symbol Connector:TestPoint
- added U?: ESP32-S3-WROOM-1U, ESP32-S3-WROOM-1U:XCVR_ESP32-S3-WROOM-1U, symbol ESP32-S3-WROOM-1U:ESP32-S3-WROOM-1U
- J?: value PowerInput5V -> PowerInput3.3V
Connections:
- net +5V is gone; now on net +3.3V: C?.1, R?.1, SW?.1 (A)
- net +3.3V: now also C?.1, J?.1 (Pin_1), U?.2 (3V3)
- net GND: now also C?.2, C?.2, C?.2, D?.1 (K), J?.1 (Pin_1), J?.1 (Pin_1), J?.1 (Pin_1), J?.2 (Pin_2), J?.4 (Pin_4), J?.4 (Pin_4), R?.2, U?.1 (GND), U?.40 (GND), U?.41_1 (GND), U?.41_2 (GND), U?.41_3 (GND), U?.41_4 (GND), U?.41_5 (GND), U?.41_6 (GND), U?.41_7 (GND), U?.41_8 (GND), U?.41_9 (GND)
- new net: J?.2 (Pin_2), SW?.2 (B)
- new net: D?.2 (A), R?.2
- new net DIR_3.3: J?.1 (Pin_1), TP?.1, U?.23 (IO21)
- new net DIR_5: J?.1 (Pin_1), J?.1 (Pin_1), TP?.1
- new net PUL_3.3: J?.2 (Pin_2), TP?.1, U?.24 (IO47)
- new net PUL_5: J?.2 (Pin_2), J?.2 (Pin_2), TP?.1
- new net Thermistor: J?.2 (Pin_2), R?.1, U?.39 (IO1)
- new net VCC: C?.1, C?.1, J?.2 (Pin_2), R?.1, SW?.1 (A), TP?.1
- no-connect marks 1 -> 9
Other:
- moved on the sheet: C?, H?, TP?
