File: PCB_v1.kicad_pcb (KiCad board)
At the start: 2 copper layers, 39 parts, among them J1 PowerInput3.3V, J10 Conn_01x20_Female, J2 PowerInput11.1V, J3 PowerOutput11.1V, J4 Thermistor, J5 LogicShifterIn, J6 LogicShifterOut, J9 Conn_01x20_Female, SW1 SW_SPDT, SW2 SW_SPDT

Commit message: completed PCB
Parts:
- removed J10: Conn_01x20_Female, Connector_PinSocket_2.54mm:PinSocket_1x20_P2.54mm_Vertical
- J9: value Conn_01x20_Female -> Conn_01x06_Female; footprint Connector_PinSocket_2.54mm:PinSocket_1x20_P2.54mm_Vertical -> Connector_PinSocket_2.54mm:PinSocket_1x06_P2.54mm_Vertical
- R3: footprint Resistor_THT:R_Axial_DIN0204_L3.6mm_D1.6mm_P2.54mm_Vertical -> Resistor_THT:R_Axial_DIN0207_L6.3mm_D2.5mm_P10.16mm_Horizontal
- moved C2 56.0 mm to (90.8, 74.2)
- moved R2 55.9 mm to (99.9, 69.7), turned to 0 degrees
- moved D2 55.7 mm to (102.5, 66.2), turned to 180 degrees
- moved J6 55.1 mm to (106.3, 102.5), turned to -90 degrees
- moved C4 51.6 mm to (90.8, 84.2)
- moved F1 50.3 mm to (117.5, 106.2)
- moved J1 46.9 mm to (92.0, 66.2), turned to 90 degrees
- moved SW2 46.4 mm to (101.0, 74.7)
- moved TP7 42.5 mm to (125.0, 70.0), turned to 180 degrees
- moved J5 42.1 mm to (106.3, 92.4), turned to -90 degrees
- moved J4 37.5 mm to (93.5, 107.5), turned to -90 degrees
- moved D1 36.0 mm to (50.0, 82.5)
- moved TP6 35.8 mm to (125.0, 75.0), turned to 180 degrees
- moved H2 32.5 mm to (135.0, 42.5)
- moved H4 32.5 mm to (135.0, 107.5)
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- renumbered PUL to J7, DIR to J8
Connections:
- J5 pad 3: unconnected-(J5-Pad3) -> +3.3V
- J6 pad 3: unconnected-(J6-Pad3) -> +5V
- J9 pad 2: unconnected-(J9-Pad2) -> /Thermistor
- J9 pad 3: unconnected-(J9-Pad3) -> /PUL_3.3
- J9 pad 4: unconnected-(J9-Pad4) -> /DIR_3.3
- J9 pad 5: unconnected-(J9-Pad5) -> GND
- J9 pad 6: unconnected-(J9-Pad6) -> +5V
Routing:
- net /DIR_5: track 0.00 -> 82.2 mm, vias 0 -> 2
- net /PUL_5: track 0.00 -> 80.5 mm
- net Net-(F1-Pad1): track 0.00 -> 66.1 mm, vias 0 -> 2
- net /PUL_3.3: track 0.00 -> 59.2 mm
- net VCC: track 0.00 -> 45.2 mm, vias 0 -> 1
- net /DIR_3.3: track 0.00 -> 45.1 mm, vias 0 -> 2
- net /Thermistor: track 0.00 -> 31.3 mm, vias 0 -> 1
- net Net-(D1-Pad2): track 0.00 -> 29.5 mm
- net Net-(F1-Pad2): track 0.00 -> 19.4 mm
- net Net-(J2-Pad2): track 0.00 -> 18.5 mm
- net +3.3V: track 0.00 -> 15.4 mm
- net Net-(D2-Pad2): track 0.00 -> 11.5 mm
- net +5V: track 0.00 -> 6.61 mm
- added copper zone on F.Cu, net +3.3V
- added copper zone on B.Cu, net GND
- added copper zone on F.Cu, net VCC
Other:
- board outline added: 92.5 x 70 mm
- board text added: "+3.3V"
- board text added: "AstraFix Desgined By: Aditya Bansal"
- board text added: "DIR"
- board text added: "DIR_3.3V"
- board text added: "DIR_5V"
- board text added: "GND"
- board text added: "HV Side"
- board text added: "LV Side"
- board text added: "PUL"
- board text added: "PUL_3.3V"
- board text added: "PUL_5V"
- board text added: "Pin 1"
- board text added: "StepperGrounds"
- board text added: "StepperSignals"
- board text added: "Ther"
- board text added: "VCC"
